File: LT8614 5V Low Noise Buck.sch (KiCad schematic (older format))
At the start: 24 parts, among them U1 LT8614EUDC

Commit message: netlist and first pcb draft
Parts:
- C1: footprint (none) -> Capacitors_SMD:c_elec_6.3x5.8
- C10, C6: footprint (none) -> Capacitors_SMD:C_1210_HandSoldering
- C11, C3: footprint (none) -> Capacitors_SMD:C_1206_HandSoldering
- C12, C13, C2, C4, C5, C7, C8, C9: footprint (none) -> Capacitors_SMD:C_0603_HandSoldering
- C14: footprint (none) -> Capacitors_SMD:C_0402
- FB1: footprint (none) -> Capacitors_SMD:C_0805
- L1: footprint (none) -> LT8614 5V Low Noise Buck:inductor-smd-2020-50x50
- L2: footprint (none) -> LT8614 5V Low Noise Buck:Inductor_Taiyo-Yuden_MD-4040
- R2, R3, R4, R5, R7: footprint (none) -> Resistors_SMD:R_0603_HandSoldering
- U1: footprint (none) -> LT8614 5V Low Noise Buck:LT8614; symbol LT8614EUDC -> LT8614EUDC-RESCUE-LT8614_5V_Low_Noise_Buck
- VOUT1: footprint (none) -> Pin_Headers:Pin_Header_Straight_1x02
Connections:
- net +24V renamed VCC
Changed lines of the file:
@@
 $EndDescr
 $Comp
-L LT8614EUDC U1
+L LT8614EUDC-RESCUE-LT8614_5V_Low_Noise_Buck U1
 U 1 1 586A3539
 P 2900 2050
 F 0 "U1" H 3700 2200 60  0000 C CNN
 F 1 "LT8614EUDC" H 3700 2100 60  0000 C CNN
-F 2 "" H 3700 2100 60  0001 C CNN
+F 2 "LT8614 5V Low Noise Buck:LT8614" H 3700 2100 60  0001 C CNN
 F 3 "" H 3650 2100 60  0001 C CNN
 	1    2900 2050
@@
 F 0 "C2" H 2525 1900 50  0000 L CNN
 F 1 "1U" H 2525 1700 50  0000 L CNN
-F 2 "" H 2538 1650 50  0000 C CNN
+F 2 "Capacitors_SMD:C_0603_HandSoldering" H 2538 1650 50  0001 C CNN
 F 3 "" H 2500 1800 50  0000 C CNN
 	1    2500 1800
@@
 F 0 "C12" H 2525 2400 50  0000 L CNN
 F 1 "1U" H 2525 2200 50  0000 L CNN
-F 2 "" H 2538 2150 50  0000 C CNN
+F 2 "Capacitors_SMD:C_0603_HandSoldering" H 2538 2150 50  0001 C CNN
 F 3 "" H 2500 2300 50  0000 C CNN
 	1    2500 2300
@@
 F 0 "C1" H 1575 1900 50  0000 L CNN
 F 1 "22U" H 1575 1700 50  0000 L CNN
-F 2 "" H 1550 1800 50  0000 C CNN
+F 2 "Capacitors_SMD:c_elec_6.3x5.8" H 1550 1800 50  0001 C CNN
 F 3 "" H 1550 1800 50  0000 C CNN
 	1    1550 1800
@@
 F 0 "C11" H 1925 1900 50  0000 L CNN
 F 1 "10U" H 1925 1700 50  0000 L CNN
-F 2 "" H 1938 1650 50  0000 C CNN
+F 2 "Capacitors_SMD:C_1206_HandSoldering" H 1938 1650 50  0001 C CNN
 F 3 "" H 1900 1800 50  0000 C CNN
 	1    1900 1800
@@
 F 0 "C7" H 2475 3100 50  0000 L CNN
 F 1 "1U" H 2475 2900 50  0000 L CNN
-F 2 "" H 2488 2850 50  0000 C CNN
+F 2 "Capacitors_SMD:C_0603_HandSoldering" H 2488 2850 50  0001 C CNN
 F 3 "" H 2450 3000 50  0000 C CNN
 	1    2450 3000
@@
 F 0 "C8" H 2925 3250 50  0000 L CNN
 F 1 "0.1U" H 2925 3050 50  0000 L CNN
-F 2 "" H 2938 3000 50  0000 C CNN
+F 2 "Capacitors_SMD:C_0603_HandSoldering" H 2938 3000 50  0001 C CNN
 F 3 "" H 2900 3150 50  0000 C CNN
 	1    2900 3150
@@
 F 0 "R2" V 3180 3350 50  0000 C CNN
 F 1 "18.2K" V 3100 3350 50  0000 C CNN
-F 2 "" V 3030 3350 50  0000 C CNN
+F 2 "Resistors_SMD:R_0603_HandSoldering" V 3030 3350 50  0001 C CNN
 F 3 "" H 3100 3350 50  0000 C CNN
 	1    3100 3350
@@
 F 0 "L2" V 5750 1500 50  0000 C CNN
 F 1 "0.22U" V 5900 1500 50  0000 C CNN
-F 2 "" H 5800 1500 50  0000 C CNN
+F 2 "LT8614 5V Low Noise Buck:Inductor_Taiyo-Yuden_MD-4040" H 5800 1500 50  0001 C CNN
 F 3 "IHLP1616ABERR22M01" V 6000 1350 50  0000 C CNN
 	1    5800 1500
@@
 F 0 "C10" H 5475 1750 50  0000 L CNN
 F 1 "10U" H 5475 1550 50  0000 L CNN
-F 2 "" H 5488 1500 50  0000 C CNN
+F 2 "Capacitors_SMD:C_1210_HandSoldering" H 5488 1500 50  0001 C CNN
 F 3 "" H 5450 1650 50  0000 C CNN
 	1    5450 1650
@@
 F 0 "C3" H 4775 1750 50  0000 L CNN
 F 1 "4.7U" H 4775 1550 50  0000 L CNN
-F 2 "" H 4788 1500 50  0000 C CNN
+F 2 "Capacitors_SMD:C_1206_HandSoldering" H 4788 1500 50  0001 C CNN
 F 3 "" H 4750 1650 50  0000 C CNN
 	1    4750 1650
@@
 F 0 "C14" H 4525 1750 50  0000 L CNN
 F 1 "0.1U" H 4525 1550 50  0000 L CNN
-F 2 "" H 4538 1500 50  0000 C CNN
+F 2 "Capacitors_SMD:C_0402" H 4538 1500 50  0001 C CNN
 F 3 "" H 4500 1650 50  0000 C CNN
 	1    4500 1650
@@
 F 0 "FB1" V 5050 1500 50  0000 C CNN
 F 1 "Ferrite Beads" V 5200 1500 50  0000 C CNN
-F 2 "" H 5100 1500 50  0000 C CNN
+F 2 "Capacitors_SMD:C_0805" H 5100 1500 50  0001 C CNN
 F 3 "810-MPZ2012S300A" V 5300 1500 50  0000 C CNN
 	1    5100 1500
@@
 F 0 "C4" H 4525 2400 50  0000 L CNN
 F 1 "0.1U" H 4525 2200 50  0000 L CNN
-F 2 "" H 4538 2150 50  0000 C CNN
+F 2 "Capacitors_SMD:C_0603_HandSoldering" H 4538 2150 50  0001 C CNN
 F 3 "" H 4500 2300 50  0000 C CNN
 	1    4500 2300
@@
 F 0 "L1" V 5100 2650 50  0000 C CNN
 F 1 "1.5U" V 4950 2650 50  0000 C CNN
-F 2 "" H 5000 2650 50  0000 C CNN
+F 2 "LT8614 5V Low Noise Buck:inductor-smd-2020-50x50" H 5000 2650 50  0001 C CNN
 F 3 "IHLP2020CZER1R5M01" V 5200 2500 50  0000 C CNN
 	1    5000 2650
@@
 F 0 "VOUT1" H 6550 2850 50  0000 C CNN
 F 1 "5V" V 6650 2700 50  0000 C CNN
-F 2 "" H 6550 2700 50  0000 C CNN
+F 2 "Pin_Headers:Pin_Header_Straight_1x02" H 6550 2700 50  0001 C CNN
 F 3 "" H 6550 2700 50  0000 C CNN
 	1    6550 2700
@@
 F 0 "C6" H 5625 2900 50  0000 L CNN
 F 1 "47U" H 5625 2700 50  0000 L CNN
-F 2 "" H 5638 2650 50  0000 C CNN
+F 2 "Capacitors_SMD:C_1210_HandSoldering" H 5638 2650 50  0001 C CNN
 F 3 "" H 5600 2800 50  0000 C CNN
 	1    5600 2800
@@
 F 0 "C13" H 5875 2900 50  0000 L CNN
 F 1 "1U" H 5875 2700 50  0000 L CNN
-F 2 "" H 5888 2650 50  0000 C CNN
+F 2 "Capacitors_SMD:C_0603_HandSoldering" H 5888 2650 50  0001 C CNN
 F 3 "" H 5850 2800 50  0000 C CNN
 	1    5850 2800
@@
 F 0 "C9" H 6125 2900 50  0000 L CNN
 F 1 "4.7U" H 6125 2700 50  0000 L CNN
-F 2 "" H 6138 2650 50  0000 C CNN
+F 2 "Capacitors_SMD:C_0603_HandSoldering" H 6138 2650 50  0001 C CNN
 F 3 "" H 6100 2800 50  0000 C CNN
 	1    6100 2800
@@
 F 0 "C5" V 5250 3450 50  0000 L CNN
 F 1 "4.7P" V 5250 3200 50  0000 L CNN
-F 2 "" H 5138 3250 50  0000 C CNN
+F 2 "Capacitors_SMD:C_0603_HandSoldering" H 5138 3250 50  0001 C CNN
 F 3 "" H 5100 3400 50  0000 C CNN
 	1    5100 3400
@@
 F 0 "R4" V 5180 3150 50  0000 C CNN
 F 1 "1M" V 5100 3150 50  0000 C CNN
-F 2 "" V 5030 3150 50  0000 C CNN
+F 2 "Resistors_SMD:R_0603_HandSoldering" V 5030 3150 50  0001 C CNN
 F 3 "" H 5100 3150 50  0000 C CNN
 	1    5100 3150
@@
 F 0 "R5" V 4630 3350 50  0000 C CNN
 F 1 "24.3K" V 4550 3350 50  0000 C CNN
-F 2 "" V 4480 3350 50  0000 C CNN
+F 2 "Resistors_SMD:R_0603_HandSoldering" V 4480 3350 50  0001 C CNN
 F 3 "" H 4550 3350 50  0000 C CNN
 	1    4550 3350
@@
 F 0 "R7" V 4530 2850 50  0000 C CNN
 F 1 "0" V 4450 2850 50  0000 C CNN
-F 2 "" V 4380 2850 50  0000 C CNN
+F 2 "Resistors_SMD:R_0603_HandSoldering" V 4380 2850 50  0001 C CNN
 F 3 "" H 4450 2850 50  0000 C CNN
 	1    4450 2850
@@
 F 0 "R3" V 4930 3000 50  0000 C CNN
 F 1 "100K" V 4850 3000 50  0000 C CNN
-F 2 "" V 4780 3000 50  0000 C CNN
+F 2 "Resistors_SMD:R_0603_HandSoldering" V 4780 3000 50  0001 C CNN
 F 3 "" H 4850 3000 50  0000 C CNN
 	1    4850 3000
@@
 Wire Wire Line
 	2500 2450 2500 2500
-$Comp
-L +24V #PWR016
-U 1 1 586BA79E
+Wire Wire Line
+	4250 1400 4250 1500
+Wire Wire Line
+	4250 1500 4800 1500
+$Comp
+L VCC #PWR016
+U 1 1 586BF5D7
 P 4250 1400
 F 0 "#PWR016" H 4250 1250 50  0001 C CNN
-F 1 "+24V" H 4250 1540 50  0000 C CNN
+F 1 "VCC" H 4250 1550 50  0000 C CNN
 F 2 "" H 4250 1400 50  0000 C CNN
 F 3 "" H 4250 1400 50  0000 C CNN
@@
 	1    0    0    -1
 $EndComp
-Wire Wire Line
-	4250 1400 4250 1500
-Wire Wire Line
-	4250 1500 4800 1500
+$Comp
+L PWR_FLAG #FLG017
+U 1 1 586BF664
+P 4500 1500
+F 0 "#FLG017" H 4500 1595 50  0001 C CNN
+F 1 "PWR_FLAG" H 4500 1680 50  0000 C CNN
+F 2 "" H 4500 1500 50  0000 C CNN
+F 3 "" H 4500 1500 50  0000 C CNN
+	1    4500 1500
+	1    0    0    -1
+$EndComp
 $EndSCHEMATC
